Commit message: Update laser_linkの追加(LiDAR用)

File: whill_description/urdf/whill_model_cr2.urdf (robot description, URDF)
Before this commit: robot whill_model_cr2, 12 links, 11 joints
Links:
- added link laser, mass 0.0001; collision box size=0.1 0.1 0.1; visual box size=0.1 0.1 0.1
Joints:
- added joint laser_joint: type fixed, parent base_link, child laser, origin xyz=0.75 0 0.05 rpy=0 -0.05235987755982989 0
